File: ATmega168P/Dev Board/devboard.brd (EAGLE design)
At the start: 50.5 x 50.8 mm, 19 parts, among them IC1 ATMEGA168-20P, IC2 7805T

Commit message: Update 1/26/16
Parts:
- removed JP3, JP4: (no value), adafruit:1X14
- removed LED1, LED2, LED3, LED4: (no value), adafruit:LED2X5
- removed PROGRAMMER, UART: 1X4-3.5MM, adafruit:1X04-3.5MM
- removed R1, R2, R3, R4: (no value), SparkFun-Passives:AXIAL-0.5
- moved IC2 25.0 mm to (34.3, 45.7), turned to 270 degrees
- moved JP1 9.67 mm to (11.4, 20.3)
- moved JP2 9.67 mm to (36.8, 20.3)
- moved C1 6.48 mm to (20.3, 45.7), turned to 270 degrees
- moved C2 5.24 mm to (15.2, 45.7), turned to 270 degrees
- moved IC1 3.81 mm to (24.1, 20.3)
- moved POWER_IN 1.27 mm to (5.08, 47.0), turned to 90 degrees
Connections:
- removed net 5V: JP1.7, JP2.6, JP3.7, JP4.6
- removed net N$2: LED2.A, R2.P$2
- removed net N$3: LED3.A, R3.P$2
- removed net N$4: LED4.A, R4.P$2
- removed net RESET: IC1.1, JP1.1, JP3.1, PROGRAMMER.4
- net GND: no longer JP3.8, JP4.8, LED1.K, LED2.K, LED3.K, LED4.K, UART.2
- net MISO: no longer JP4.4, PROGRAMMER.2
- net MOSI: no longer JP4.3, PROGRAMMER.1
- net N$1: now also IC1.1, JP1.1; no longer LED1.A, R1.P$2
- net PIN10: no longer JP3.10
- net PIN11: no longer JP3.11
- net PIN12: no longer JP3.12
- net PIN13: no longer JP3.13
- net PIN14: no longer JP3.14
- net PIN15: no longer JP4.1
- net PIN16: no longer JP4.2
- net PIN2: no longer JP3.2, UART.3
- net PIN21: no longer JP4.7
- net PIN23: no longer JP4.9, R1.P$1
- net PIN24: no longer JP4.10, R2.P$1
- net PIN25: no longer JP4.11, R3.P$1
- net PIN26: no longer JP4.12, R4.P$1
- net PIN27: no longer JP4.13
- net PIN28: no longer JP4.14
- net PIN3: no longer JP3.3, UART.4
- net PIN4: no longer JP3.4
- net PIN5: no longer JP3.5
- net PIN6: no longer JP3.6
- net PIN9: no longer JP3.9
- net SCK: no longer JP4.5, PROGRAMMER.3
- net VCC: now also JP1.7, JP2.6; no longer UART.1
Routing:
- net 5V: track 50.7 -> 0.00 mm
- net PIN24: track 46.6 -> 0.00 mm
- net PIN23: track 46.3 -> 0.00 mm, vias 1 -> 0
- net RESET: track 46.1 -> 0.00 mm, vias 1 -> 0
- net PIN25: track 44.0 -> 0.00 mm, vias 1 -> 0
- net PIN2: track 43.7 -> 0.00 mm
- net VCC: track 78.2 -> 35.6 mm, vias 1 -> 0
- net PIN26: track 42.2 -> 0.00 mm
- net PIN3: track 35.1 -> 0.00 mm
- net N$3: track 32.1 -> 0.00 mm
- net N$2: track 27.3 -> 0.00 mm
- net N$1: track 25.0 -> 0.00 mm
- net PIN11: track 22.5 -> 0.00 mm
- net MOSI: track 21.6 -> 0.00 mm
- net PIN21: track 21.1 -> 0.00 mm
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Other:
- board text added: "G"
