File: ATmega168P/Dev Board/devboard.sch (EAGLE design)
At the start: 19 parts, among them IC1 ATMEGA168-20P, IC2 7805T

Commit message: Update 1/26/16
Parts:
- removed JP3, JP4: (no value), adafruit:PINHD-1X14
- removed LED1, LED2, LED3, LED4: (no value), adafruit:LEDSQR2X5
- removed PROGRAMMER, UART: 1X4-3.5MM, adafruit:1X4-3.5MM
- removed R1, R2, R3, R4: (no value), SparkFun-Passives:RESISTORPTH-1/2W
Connections:
- removed net 5V: JP1.7, JP2.6, JP3.7, JP4.6
- removed net N$2: LED2.A, R2.2
- removed net N$3: LED3.A, R3.2
- removed net N$4: LED4.A, R4.2
- removed net RESET: IC1.PC6(/RESET/PCI14), JP1.1, JP3.1, PROGRAMMER.4
- net GND: no longer JP3.8, JP4.8, LED1.C, LED2.C, LED3.C, LED4.C, UART.2
- net MISO: no longer JP4.4, PROGRAMMER.2
- net MOSI: no longer JP4.3, PROGRAMMER.1
- net N$1: now also IC1.PC6(/RESET/PCI14), JP1.1; no longer LED1.A, R1.2
- net PIN10: no longer JP3.10
- net PIN11: no longer JP3.11
- net PIN12: no longer JP3.12
- net PIN13: no longer JP3.13
- net PIN14: no longer JP3.14
- net PIN15: no longer JP4.1
- net PIN16: no longer JP4.2
- net PIN2: no longer JP3.2, UART.3
- net PIN21: no longer JP4.7
- net PIN23: no longer JP4.9, R1.1
- net PIN24: no longer JP4.10, R2.1
- net PIN25: no longer JP4.11, R3.1
- net PIN26: no longer JP4.12, R4.1
- net PIN27: no longer JP4.13
- net PIN28: no longer JP4.14
- net PIN3: no longer JP3.3, UART.4
- net PIN4: no longer JP3.4
- net PIN5: no longer JP3.5
- net PIN6: no longer JP3.6
- net PIN9: no longer JP3.9
- net SCK: no longer JP4.5, PROGRAMMER.3
- net VCC: now also JP1.7, JP2.6; no longer UART.1
Other:
- note removed: "When using Arduino as programmer, use the Arduino to power the board as well."
- moved on the sheet: JP1, JP2
