File: Nordic nrf51/RobotVac/robot_vac.brd (EAGLE design)
At the start: 53.3 x 52.1 mm, 22 parts, among them IC4 317T, IC5 LM340H-05, J1 1X2-3.5MM, J2 ARDUINO_R3_SHIELDNOLABELS, X1 HD44780LCD-1602

Commit message: Update 1/26/16
Parts:
- removed C3: 1uF, SparkFun-Capacitors:CAP-PTH-SMALL
- removed D1, D2: 1N4004, adafruit:DO41-10
- removed IC4: 317T, linear:TO220H
- removed R1: 400ohm, SparkFun-Passives:AXIAL-0.5
- removed R2: 240ohm, SparkFun-Passives:AXIAL-0.5
- added H_BRIDGE: SN75441_H_BRIDGE, max parts:DIL16
- added IC1: LD117AS18TR, v-reg:SOT223
- JP1: value Left Servo -> Left Motor; device adafruit:1X03 -> SparkFun-Connectors:1X02_LOCK
- JP2: value Right Servo -> Right Motor; device adafruit:1X03 -> SparkFun-Connectors:1X02_LOCK
- moved C1 25.0 mm to (34.3, 43.2), turned to 90 degrees
- moved IC5 16.2 mm to (22.9, 44.5)
- moved C2 12.8 mm to (16.5, 34.3)
- moved C4 12.7 mm to (12.7, 34.3)
- moved TM1 6.48 mm to (43.2, 20.3)
- moved JP1 5.08 mm to (45.7, 27.9)
- moved JP2 1.27 mm to (7.62, 20.3), turned to 90 degrees
Connections:
- removed net N$3: C3.1, D2.A, IC4.1, R1.P$2, R2.P$1
- removed net SERVO_LEFT: J2.D10, JP1.2
- removed net SERVO_RIGHT: J2.D11, JP2.2
- new net /MOTOR_LEFT_FWRD: H_BRIDGE.2, J2.D10
- new net /MOTOR_LEFT_REVERSE: H_BRIDGE.7, J2.SDA
- new net /MOTOR_RIGHT_FWRD: H_BRIDGE.15, J2.D11
- new net /MOTOR_RIGHT_REVERSE: H_BRIDGE.10, J2.SCL
- new net BLACK_L: H_BRIDGE.3, JP1.1
- new net BLACK_R: H_BRIDGE.11, JP2.2
- new net RED_L: H_BRIDGE.6, JP1.2
- new net RED_R: H_BRIDGE.14, JP2.1
- net 3.3V: now also IC1.4; no longer D1.A, D2.C, IC4.2, R2.P$2
- net 5V: now also H_BRIDGE.1, H_BRIDGE.16, H_BRIDGE.9
- net GND: now also H_BRIDGE.12, H_BRIDGE.13, H_BRIDGE.4, H_BRIDGE.5, IC1.1; no longer C3.2, JP1.3, JP2.3, R1.P$1
- net VCC: now also H_BRIDGE.8, IC1.3; no longer D1.C, IC4.3, JP1.1, JP2.1
Routing:
- net SERVO_LEFT: track 66.6 -> 0.00 mm
- net /MOTOR_RIGHT_REVERSE: track 0.00 -> 45.1 mm
- net VCC: track 94.7 -> 58.4 mm
- net N$3: track 35.6 -> 0.00 mm
- net /MOTOR_LEFT_REVERSE: track 0.00 -> 34.7 mm
- net BLACK_R: track 0.00 -> 33.5 mm
- net 3.3V: track 97.9 -> 67.1 mm, vias 2 -> 1
- net BLACK_L: track 0.00 -> 24.9 mm
- net LCD_RS: track 45.3 -> 65.3 mm, vias 2 -> 0
- net /MOTOR_RIGHT_FWRD: track 0.00 -> 19.9 mm
- net /MOTOR_LEFT_FWRD: track 0.00 -> 19.9 mm
- net RED_R: track 0.00 -> 19.6 mm
- net RED_L: track 0.00 -> 18.5 mm
- net 5V: track 109.5 -> 125.5 mm
- net LCD_E: track 48.2 -> 57.5 mm, vias 1 -> 0
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Other:
- board text added: "+"
- board text added: "-"
- board text added: "BLACK"
- board text added: "P0.01"
- board text added: "P0.06"
- board text added: "P0.07"
- board text added: "RED"
